Commit message: [Feature] Touch Sensor

File: mujoco_ros2_control_demos/urdf/test_vertical_cart_velocity_pid.xacro.urdf (robot description, URDF)
Before this commit: robot cart, 3 links, 2 joints
Joints:
- joint slider_to_cart: limit lower=-2.5 upper=2.5 effort=1000.0 velocity=30 -> lower=-100 upper=100 effort=1000.0 velocity=30
