Commit message: Fix reset simulation service for robots using PID control (#140)

File: mujoco_ros2_control_demos/demo_resources/robot/test_robot.urdf (robot description, URDF)
Before this commit: robot two_dof_robot, 13 links, 12 joints
Joints:
- joint joint1: axis 0 0 1 -> 0 1 0
- joint joint2: axis 0 0 1 -> 0 1 0
